Commit message: Adjusted angle limitations on the head_to_base_link joint

File: urdf/ptbr.xacro (robot description, xacro)
@@ -129,5 +129,5 @@
   <child link="head_1"/>
   <axis xyz="1.0 0.0 -0.0"/>
-  <limit upper="-2.356194" lower="-3.926991" effort="100" velocity="100"/>
+  <limit upper="0.785399" lower="-0.785399" effort="100" velocity="100"/>
 </joint>
 <joint name="right_wheel_to_base_link" type="continuous">

Commit message: fixed urdf launchfile, finished urdf

File: urdf/ptbr.xacro (robot description, xacro)
@@ -45,7 +45,7 @@
   </collision>
 </link>
-<joint name="head_to_base" type="revolute">
+<joint name="head_link" type="revolute">
   <origin xyz="0 -0.0327525 0.085" rpy="0 0 0"/>
-  <parent link="base"/>
+  <parent link="base_link"/>
   <child link="head"/>
   <axis xyz="1.0 0.0 0.0"/>
@@ -90,6 +90,24 @@
     </geometry>
   </collision>
-</link>
-<joint name="camera_to_head" type="fixed">
+  <collision>
+    <origin xyz="0 0.041 0.138" rpy="0.0 0.0 0.0"/>
+    <geometry>
+      <box size="0.106 0.018 0.106"/>
+    </geometry>
+  </collision>
+  <collision>
+    <origin xyz="0 0 0.024" rpy="0.0 0.0 0.0"/>
+    <geometry>
+      <box size="0.038895 0.038895 0.048"/>
+    </geometry>
+  </collision>
+  <collision>
+    <origin xyz="0.0 0.0 0.068" rpy="0.0 0.0 0.0"/>
+    <geometry>
+      <box size="0.0525 0.0525 0.04"/>
+    </geometry>
+  </collision>
+</link>
+<joint name="camera_joint" type="fixed">
   <origin xyz="0.0 0.051235 0.174" rpy="0.0 0.0 0.0"/>
   <parent link="head"/>
@@ -164,5 +182,11 @@
   </collision>
 </link>
-<link name="left_arm_1">
+<joint name="left_arm_joint" type="continuous">
+  <origin xyz="-0.05 0.0 0.146862" rpy="0 -${pi/2} 0"/>
+  <parent link="head"/>
+  <child link="left_arm"/>
+  <axis xyz="0 0.0 -1"/>
+</joint>
+<link name="left_arm">
   <inertial>
     <origin xyz="0.018087977944126324 -0.005800896128886866 -0.056698307724850905" rpy="0 0 0"/>
@@ -171,18 +195,24 @@
   </inertial>
   <visual>
-    <origin xyz="-0.049692 -0.041636 -0.266278" rpy="0 0 0"/>
-    <geometry>
-      <mesh filename="file://$(find ptbr)/meshes/left_arm_1.stl" scale="0.001 0.001 0.001"/>
-    </geometry>
-    <material name="silver"/>
-  </visual>
-  <collision>
-    <origin xyz="-0.049692 -0.041636 -0.266278" rpy="0 0 0"/>
-    <geometry>
-      <mesh filename="file://$(find ptbr)/meshes/left_arm_1.stl" scale="0.001 0.001 0.001"/>
-    </geometry>
-  </collision>
-</link>
-<link name="right_arm_1">
+    <origin xyz="-0.266278 0.041636 -0.049692" rpy="${pi} -${pi/2} 0"/>
+    <geometry>
+      <mesh filename="package://ptbr/meshes/left_arm_1.stl" scale="0.001 0.001 0.001"/>
+    </geometry>
+    <material name="silver"/>
+  </visual>
+  <collision>
+    <origin xyz="-0.266278 0.041636 -0.049692" rpy="${pi} -${pi/2} 0"/>
+    <geometry>
+      <mesh filename="package://ptbr/meshes/left_arm_1.stl" scale="0.001 0.001 0.001"/>
+    </geometry>
+  </collision>
+</link>
+<joint name="right_arm_joint" type="continuous">
+  <origin xyz="0.05 0.0 0.146862" rpy="0 ${pi/2} 0"/>
+  <parent link="head"/>
+  <child link="right_arm"/>
+  <axis xyz="0 0.0 1"/>
+</joint>
+<link name="right_arm">
   <inertial>
     <origin xyz="-0.018087407770600646 -0.005810132869209922 -0.056697751450645734" rpy="0 0 0"/>
@@ -191,28 +221,16 @@
   </inertial>
   <visual>
-    <origin xyz="0.050308 -0.041636 -0.266278" rpy="0 0 0"/>
-    <geometry>
-      <mesh filename="file://$(find ptbr)/meshes/right_arm_1.stl" scale="0.001 0.001 0.001"/>
-    </geometry>
-    <material name="silver"/>
-  </visual>
-  <collision>
-    <origin xyz="0.050308 -0.041636 -0.266278" rpy="0 0 0"/>
-    <geometry>
-      <mesh filename="file://$(find ptbr)/meshes/right_arm_1.stl" scale="0.001 0.001 0.001"/>
-    </geometry>
-  </collision>
-</link>
-<joint name="left_arm_to_base_link" type="continuous">
-  <origin xyz="0.05 0.0 0.146862" rpy="0 0 0"/>
-  <parent link="head"/>
-  <child link="left_arm_1"/>
-  <axis xyz="1.0 0.0 -0.0"/>
-</joint>
-<joint name="right_arm_to_base_link" type="continuous">
-  <origin xyz="-0.05 0.0 0.146862" rpy="0 0 0"/>
-  <parent link="head"/>
-  <child link="right_arm_1"/>
-  <axis xyz="-1.0 -0.0 0.0"/>
-</joint>
+    <origin xyz="0.266278 0.041636 -0.050308" rpy="${pi} ${pi/2} 0"/>
+    <geometry>
+      <mesh filename="package://ptbr/meshes/right_arm_1.stl" scale="0.001 0.001 0.001"/>
+    </geometry>
+    <material name="silver"/>
+  </visual>
+  <collision>
+    <origin xyz="0.266278 0.041636 -0.050308" rpy="${pi} ${pi/2} 0"/>
+    <geometry>
+      <mesh filename="package://ptbr/meshes/right_arm_1.stl" scale="0.001 0.001 0.001"/>
+    </geometry>
+  </collision>
+</link>
 </robot>

Commit message: SLAM on battery, start on gazebo

File: urdf/ptbr.xacro (robot description, xacro)
@@ -4,4 +4,5 @@
 <xacro:include filename="$(find ptbr)/urdf/ptbr.ros2control" />
 <xacro:include filename="$(find ptbr)/urdf/ptbr.gazebo" />
+<xacro:include filename="$(find ptbr)/urdf/camera.xacro" />
 <link name="base_link">
 </link>
@@ -109,25 +110,4 @@
   </collision>
 </link>
-<joint name="camera_joint" type="fixed">
-  <origin xyz="0.0 0.051235 0.174" rpy="0.0 0.0 0.0"/>
-  <parent link="head"/>
-  <child link="camera_link"/>
-  <axis xyz="0.0 0.0 0.0"/>
-</joint>
-<link name="camera_link">
-  <visual>
-    <origin xyz="0.0 0.0 0.0" rpy="0.0 0.0 0.0"/>
-    <geometry>
-      <box size="0.09093 0.00247 0.027965"/>
-    </geometry>
-    <material name="red"/>
-  </visual>
-  <collision>
-    <origin xyz="0.0 0.0 0.0" rpy="0.0 0.0 0.0"/>
-    <geometry>
-      <box size="0.09093 0.00247 0.027965"/>
-    </geometry>
-  </collision>
-</link>
 <joint name="right_wheel_joint" type="continuous">
   <origin xyz="0.06 0 0" rpy="0 ${pi/2} 0"/>
@@ -135,4 +115,6 @@
   <child link="right_wheel"/>
   <axis xyz="0 0.0 -1"/>
+  <limit effort="50000" velocity="10"/>
+  <dynamics damping="1.0" friction="1.0"/>
 </joint>
 <link name="right_wheel">
@@ -161,4 +143,6 @@
   <child link="left_wheel"/>
   <axis xyz="0 0.0 1"/>
+  <limit effort="50000" velocity="10"/>
+  <dynamics damping="1.0" friction="1.0"/>
 </joint>
 <link name="left_wheel">

Commit message: gazebo

File: urdf/ptbr.xacro (robot description, xacro)
@@ -46,5 +46,5 @@
   </collision>
 </link>
-<joint name="head_link" type="revolute">
+<joint name="head_joint" type="revolute">
   <origin xyz="0 -0.0327525 0.085" rpy="0 0 0"/>
   <parent link="base_link"/>

Commit message: gazebo FIXED
HELL YEAH

File: urdf/ptbr.xacro (robot description, xacro)
@@ -14,5 +14,5 @@
   <inertial>
     <origin xyz="-0.00030771491577107806 0.006425674318858227 0.038113735190444614" rpy="0 0 0"/>
-    <mass value="6.4013846052337655"/>
+    <mass value="10"/>
     <inertia ixx="0.018437" iyy="0.007171" izz="0.017545" ixy="0.0" iyz="-0.001397" ixz="-0.0"/>
   </inertial>
@@ -56,5 +56,5 @@
   <inertial>
     <origin xyz="2.850842288221471e-07 -0.001985837786485485 0.12158816571318953" rpy="0 0 0"/>
-    <mass value="9.976187828305356"/>
+    <mass value="2"/>
     <inertia ixx="0.029478" iyy="0.029097" izz="0.015168" ixy="0.0" iyz="0.000325" ixz="-0.0"/>
   </inertial>
@@ -121,5 +121,5 @@
   <inertial>
     <origin xyz="-0.019999714915771002 -2.0220914574015092e-07 2.2264549151551627e-07" rpy="0 0 0"/>
-    <mass value="1.1403478677706373"/>
+    <mass value="1"/>
     <inertia ixx="0.000659" iyy="0.000482" izz="0.000482" ixy="0.0" iyz="0.0" ixz="-0.0"/>
   </inertial>
@@ -149,5 +149,5 @@
   <inertial>
     <origin xyz="-0.019999714915771002 -2.0220914574015092e-07 2.2264549151551627e-07" rpy="0 0 0"/>
-    <mass value="1.1403478677706373"/>
+    <mass value="1"/>
     <inertia ixx="0.000659" iyy="0.000482" izz="0.000482" ixy="0.0" iyz="0.0" ixz="-0.0"/>
   </inertial>
@@ -175,5 +175,5 @@
   <inertial>
     <origin xyz="0.018087977944126324 -0.005800896128886866 -0.056698307724850905" rpy="0 0 0"/>
-    <mass value="1.013009141787747"/>
+    <mass value="0.1"/>
     <inertia ixx="0.002313" iyy="0.002182" izz="0.000268" ixy="8e-06" iyz="-0.00039" ixz="6.4e-05"/>
   </inertial>
@@ -201,5 +201,5 @@
   <inertial>
     <origin xyz="-0.018087407770600646 -0.005810132869209922 -0.056697751450645734" rpy="0 0 0"/>
-    <mass value="1.0130091381540007"/>
+    <mass value="0.1"/>
     <inertia ixx="0.002313" iyy="0.002182" izz="0.000268" ixy="-8e-06" iyz="-0.00039" ixz="-6.4e-05"/>
   </inertial>
