Commit message: Flipped the entire moddel, NAV2 (still, this is bad)

File: urdf/camera.xacro (robot description, xacro)
@@ -2,5 +2,5 @@
 <robot xmlns:xacro="http://www.ros.org/wiki/xacro" >
     <joint name="camera_joint" type="fixed">
-        <origin xyz="0.0 0.051235 0.176" rpy="0.0 0.0 ${pi/2}"/>
+        <origin xyz="0.051235 0.0 0.176" rpy="0.0 0.0 0"/>
         <parent link="head"/>
         <child link="camera_link"/>

File: urdf/ptbr.xacro (robot description, xacro)
@@ -5,4 +5,11 @@
 <xacro:include filename="$(find ptbr)/urdf/ptbr.gazebo" />
 <xacro:include filename="$(find ptbr)/urdf/camera.xacro" />
+<link name="base_footprint">
+</link>
+<joint name="base_link_joint" type="fixed">
+  <origin xyz="0 0 0.0325"/>
+  <parent link="base_footprint"/>
+  <child link="base_link"/>
+</joint>
 <link name="base_link">
 </link>
@@ -13,5 +20,5 @@
 <link name="base">
   <inertial>
-    <origin xyz="-0.00030771491577107806 0.006425674318858227 0.038113735190444614" rpy="0 0 0"/>
+    <origin xyz="0.006425674318858227 -0.00030771491577107806 0.038113735190444614" rpy="0 0 0"/>
     <mass value="10"/>
     <inertia ixx="0.018437" iyy="0.007171" izz="0.017545" ixy="0.0" iyz="-0.001397" ixz="-0.0"/>
@@ -20,10 +27,10 @@
     <origin xyz="0 0 0.006" rpy="0 0 0"/>
     <geometry>
-      <box size="0.08 0.1634 0.06"/>
-    </geometry>
-    <material name="silver"/>
-  </visual>
-  <visual>
-    <origin xyz="0.0 -0.0327525 0.0575" rpy="0.0 0.0 0.0"/>
+      <box size="0.1634 0.08 0.06"/>
+    </geometry>
+    <material name="silver"/>
+  </visual>
+  <visual>
+    <origin xyz="-0.0327525 0.0 0.0575" rpy="0.0 0.0 0.0"/>
     <geometry>
       <box size="0.032895 0.032895 0.055"/>
@@ -34,10 +41,10 @@
     <origin xyz="0 0 0.006" rpy="0 0 0"/>
     <geometry>
-      <box size="0.08 0.1634 0.06"/>
-    </geometry>
-    <material name="silver"/>
-  </collision>
-  <collision>
-    <origin xyz="0.0 -0.0327525 0.0575" rpy="0.0 0.0 0.0"/>
+      <box size="0.1634 0.08 0.06"/>
+    </geometry>
+    <material name="silver"/>
+  </collision>
+  <collision>
+    <origin xyz="-0.0327525 0.0 0.0575" rpy="0.0 0.0 0.0"/>
     <geometry>
       <box size="0.032895 0.032895 0.055"/>
@@ -47,8 +54,8 @@
 </link>
 <joint name="head_joint" type="revolute">
-  <origin xyz="0 -0.0327525 0.085" rpy="0 0 0"/>
+  <origin xyz="-0.0327525 0 0.085" rpy="0 0 0"/>
   <parent link="base_link"/>
   <child link="head"/>
-  <axis xyz="1.0 0.0 0.0"/>
+  <axis xyz="0.0 1.0 0.0"/>
   <limit upper="0.785399" lower="-0.785399" effort="100" velocity="100"/>
 </joint>
@@ -67,7 +74,7 @@
   </visual>
   <visual>
-    <origin xyz="0 0.041 0.138" rpy="0.0 0.0 0.0"/>
-    <geometry>
-      <box size="0.106 0.018 0.106"/>
+    <origin xyz="0.041 0 0.138" rpy="0.0 0.0 0.0"/>
+    <geometry>
+      <box size="0.018 0.106 0.106"/>
     </geometry>
   </visual>
@@ -92,7 +99,7 @@
   </collision>
   <collision>
-    <origin xyz="0 0.041 0.138" rpy="0.0 0.0 0.0"/>
-    <geometry>
-      <box size="0.106 0.018 0.106"/>
+    <origin xyz="0.041 0 0.138" rpy="0.0 0.0 0.0"/>
+    <geometry>
+      <box size="0.018 0.106 0.106"/>
     </geometry>
   </collision>
@@ -111,5 +118,5 @@
 </link>
 <joint name="right_wheel_joint" type="continuous">
-  <origin xyz="0.06 0 0" rpy="0 ${pi/2} 0"/>
+  <origin xyz="0 -0.06 0" rpy="${pi/2} 0 0"/>
   <parent link="base_link"/>
   <child link="right_wheel"/>
@@ -139,5 +146,5 @@
 </link>
 <joint name="left_wheel_joint" type="continuous">
-  <origin xyz="-0.06 0 0" rpy="0 -${pi/2} 0"/>
+  <origin xyz="0 0.06 0" rpy="-${pi/2} 0 0"/>
   <parent link="base_link"/>
   <child link="left_wheel"/>
@@ -167,5 +174,5 @@
 </link>
 <joint name="left_arm_joint" type="continuous">
-  <origin xyz="-0.05 0.0 0.146862" rpy="0 -${pi/2} 0"/>
+  <origin xyz="0.0 0.05 0.146862" rpy="-${pi/2} 0 0"/>
   <parent link="head"/>
   <child link="left_arm"/>
@@ -179,5 +186,5 @@
   </inertial>
   <visual>
-    <origin xyz="-0.266278 0.041636 -0.049692" rpy="${pi} -${pi/2} 0"/>
+    <origin xyz="0.041636 0.266278 -0.049692" rpy="-${pi/2} -${pi/2} ${pi}"/>
     <geometry>
       <mesh filename="package://ptbr/meshes/left_arm_1.stl" scale="0.001 0.001 0.001"/>
@@ -186,5 +193,5 @@
   </visual>
   <collision>
-    <origin xyz="-0.266278 0.041636 -0.049692" rpy="${pi} -${pi/2} 0"/>
+    <origin xyz="0.041636 0.266278 -0.049692" rpy="-${pi/2} -${pi/2} ${pi}"/>
     <geometry>
       <mesh filename="package://ptbr/meshes/left_arm_1.stl" scale="0.001 0.001 0.001"/>
@@ -193,5 +200,5 @@
 </link>
 <joint name="right_arm_joint" type="continuous">
-  <origin xyz="0.05 0.0 0.146862" rpy="0 ${pi/2} 0"/>
+  <origin xyz="0.0 -0.05 0.146862" rpy="${pi/2} 0 0"/>
   <parent link="head"/>
   <child link="right_arm"/>
@@ -205,5 +212,5 @@
   </inertial>
   <visual>
-    <origin xyz="0.266278 0.041636 -0.050308" rpy="${pi} ${pi/2} 0"/>
+    <origin xyz="0.041636 -0.266278 -0.050308" rpy="${pi/2} ${pi/2} ${pi}"/>
     <geometry>
       <mesh filename="package://ptbr/meshes/right_arm_1.stl" scale="0.001 0.001 0.001"/>
@@ -212,5 +219,5 @@
   </visual>
   <collision>
-    <origin xyz="0.266278 0.041636 -0.050308" rpy="${pi} ${pi/2} 0"/>
+    <origin xyz="0.041636 -0.266278 -0.050308" rpy="${pi/2} ${pi/2} ${pi}"/>
     <geometry>
       <mesh filename="package://ptbr/meshes/right_arm_1.stl" scale="0.001 0.001 0.001"/>
